Commit message: mmm

File: controllers/generic_inverse_kinematic/filename1.urdf (robot description, URDF)
Before this commit: robot UR3e, 7 links, 5 joints
Links:
- removed link forearm_link
- removed link shoulder_link
- removed link upper_arm_link
- removed link wrist_1_link
- removed link wrist_2_link
- removed link wrist_3_joint
- added link LINK_1; collision cylinder length=0.063 radius=0.0225; collision sphere radius=0.0225
- added link LINK_2; collision cylinder length=0.336 radius=0.0225; collision sphere radius=0.0225
- added link LINK_3; collision cylinder length=0.186 radius=0.0225; collision sphere radius=0.0225
- added link LINK_4; collision cylinder length=0.334 radius=0.0225; collision sphere radius=0.0225
- added link LINK_5; collision cylinder length=0.04 radius=0.0225; collision sphere radius=0.0225
- added link LINK_6; collision box size=0.25 0.02 0.06; collision cylinder length=0.032 radius=0.0225
- added link camera
- added link ds_left
- added link ds_right
- link base_link: geometry collision box size=0.31 0.15 0.35; collision cylinder length=0.1 radius=0.05
Joints:
- removed joint elbow_joint
- removed joint shoulder_lift_joint
- removed joint shoulder_pan_joint
- removed joint wrist_1_joint
- removed joint wrist_2_joint
- added joint base_link_camera_joint: type fixed, parent base_link, child camera, origin xyz=-9.28752e-07 0 0.35 rpy=3.1415927 2.6535897e-06 3.1415927
- added joint base_link_ds_left_joint: type fixed, parent base_link, child ds_left, origin xyz=0.07 0.055 0.34 rpy=0 -1.0089953 0
- added joint base_link_ds_right_joint: type fixed, parent base_link, child ds_right, origin xyz=-0.07 0 0.34 rpy=3.1415927 -1.0471973 3.1415927
- added joint joint_1_motor: type revolute, parent base_link, child LINK_1, origin xyz=0 0.075 0.3 rpy=0 0 0, axis 0 1 0, limit lower=-6 upper=6 effort=10 velocity=10
- added joint joint_2_motor: type revolute, parent LINK_1, child LINK_2, origin xyz=0 0.04 0 rpy=0 0 0, axis 1 0 0, limit lower=-6 upper=6 effort=10 velocity=10
- added joint joint_3_motor: type revolute, parent LINK_2, child LINK_3, origin xyz=0 0.324 0 rpy=0 0 0, axis 1 0 0, limit lower=-6 upper=6 effort=10 velocity=10
- added joint joint_4_motor: type revolute, parent LINK_3, child LINK_4, origin xyz=0 0.174 0 rpy=0 0 0, axis 1 0 0, limit lower=-6 upper=6 effort=10 velocity=10
- added joint joint_5_motor: type revolute, parent LINK_4, child LINK_5, origin xyz=0 0.324 0 rpy=0 0 0, axis 0 1 0, limit lower=-6 upper=6 effort=10 velocity=10
- added joint joint_6_motor: type revolute, parent LINK_5, child LINK_6, origin xyz=0 0.03 0 rpy=0 0 0, axis 1 0 0, limit lower=-6 upper=6 effort=10 velocity=10

Commit message: kinematics

File: controllers/generic_inverse_kinematic/filename1.urdf (robot description, URDF)
Before this commit: robot robot, 10 links, 9 joints
Links:
- removed link LINK_1
- removed link LINK_2
- removed link LINK_3
- removed link LINK_4
- removed link LINK_5
- removed link LINK_6
- removed link camera
- removed link ds_left
- removed link ds_right
- added link forearm_link; collision cylinder length=0.05 radius=0.037; collision cylinder length=0.1 radius=0.03
- added link shoulder_link; collision cylinder length=0.066 radius=0.045; collision cylinder length=0.121 radius=0.046
- added link upper_arm_link; collision cylinder length=0.073 radius=0.046; collision cylinder length=0.11 radius=0.038
- added link wrist_1_link; collision cylinder length=0.064 radius=0.032; collision cylinder length=0.1 radius=0.033
- added link wrist_2_link; collision cylinder length=0.043 radius=0.032; collision cylinder length=0.097 radius=0.032
- added link wrist_3_joint
- link base_link: geometry collision cylinder length=0.09 radius=0.064; visual cylinder length=0.09 radius=0.064
Joints:
- removed joint base_link_camera_joint
- removed joint base_link_ds_left_joint
- removed joint base_link_ds_right_joint
- removed joint joint_1_motor
- removed joint joint_2_motor
- removed joint joint_3_motor
- removed joint joint_4_motor
- removed joint joint_5_motor
- removed joint joint_6_motor
- added joint elbow_joint: type revolute, parent upper_arm_link, child forearm_link, origin xyz=0 -0.093 0.244 rpy=0 0 0, axis 0 1 0, limit lower=-3.14159 upper=3.14159 effort=150 velocity=3.14
- added joint shoulder_lift_joint: type revolute, parent shoulder_link, child upper_arm_link, origin xyz=0 0.12 0 rpy=0 1.570796 0, axis 0 1 0, limit lower=-6.28319 upper=6.28319 effort=330 velocity=3.14
- added joint shoulder_pan_joint: type revolute, parent base_link, child shoulder_link, origin xyz=0 0 0.152 rpy=0 0 0, axis 0 0 1, limit lower=-6.28319 upper=6.28319 effort=330 velocity=3.14
- added joint wrist_1_joint: type revolute, parent forearm_link, child wrist_1_link, origin xyz=0 0 0.213 rpy=0 1.570796 0, axis 0 1 0, limit lower=-6.28319 upper=6.28319 effort=54 velocity=6.28
- added joint wrist_2_joint: type revolute, parent wrist_1_link, child wrist_2_link, origin xyz=0 0.104 0 rpy=0 0 0, axis 0 0 1, limit lower=-6.28319 upper=6.28319 effort=54 velocity=6.28
